File: pcbs/biking_leds.kicad_pcb (KiCad board)
At the start: 2 copper layers, 33.5 x 64 mm, 10 parts, among them U1 ATtiny1616-S, U2 TMF8820

Commit message: Add files via upload
Other:
- board text added: "Shelley Ma #Falling Out"
Changed lines of the file:
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@@
 		(layer "Edge.Cuts")
+	)
+	(gr_text "Shelley Ma\n#Falling Out"
+		(at 114.23 91.5 0)
+		(layer "F.SilkS")
+		(effects
+			(font
+				(size 1 1)
+				(thickness 0.15)
+			)
+			(justify left bottom)
+		)
+	)
+	(segment
+		(start 99.5 60.5)
+		(end 99.5 57.710001)
+		(width 0.25)
+		(layer "F.Cu")
+		(net "+3V3")
+	)
+	(segment
+		(start 100.634092 73)
+		(end 96 68.365908)
+		(width 0.25)
+		(layer "F.Cu")
+		(net "+3V3")
+	)
+	(segment
+		(start 105.1 71.64)
+		(end 105.1 65.6)
+		(width 0.25)
+		(layer "F.Cu")
+		(net "+3V3")
+	)
+	(segment
+		(start 99.5 57.710001)
+		(end 98.869999 57.08)
+		(width 0.25)
+		(layer "F.Cu")
+		(net "+3V3")
+	)
+	(segment
+		(start 96 68.365908)
+		(end 96 57)
+		(width 0.25)
+		(layer "F.Cu")
+		(net "+3V3")
+	)
+	(segment
+		(start 105.1 65.6)
+		(end 100 60.5)
+		(width 0.25)
+		(layer "F.Cu")
+		(net "+3V3")
+	)
+	(segment
+		(start 100 60.5)
+		(end 99.5 60.5)
+		(width 0.25)
+		(layer "F.Cu")
+		(net "+3V3")
+	)
+	(segment
+		(start 96.08 57.08)
+		(end 97.845 57.08)
+		(width 0.25)
+		(layer "F.Cu")
+		(net "+3V3")
+	)
+	(segment
+		(start 101 73)
+		(end 100.634092 73)
+		(width 0.25)
+		(layer "F.Cu")
+		(net "+3V3")
+	)
+	(segment
+		(start 96 57)
+		(end 96.08 57.08)
+		(width 0.25)
+		(layer "F.Cu")
+		(net "+3V3")
+	)
+	(segment
+		(start 98.869999 57.08)
+		(end 97.845 57.08)
+		(width 0.25)
+		(layer "F.Cu")
+		(net "+3V3")
+	)
+	(segment
+		(start 101 63.020001)
+		(end 98.869999 60.89)
+		(width 0.25)
+		(layer "F.Cu")
+		(net "Net-(U1-PA6)")
+	)
+	(segment
+		(start 101 71.64)
+		(end 101 63.020001)
+		(width 0.25)
+		(layer "F.Cu")
+		(net "Net-(U1-PA6)")
+	)
+	(segment
+		(start 98.869999 60.89)
+		(end 97.845 60.89)
+		(width 0.25)
+		(layer "F.Cu")
+		(net "Net-(U1-PA6)")
 	)
 	(via
@@
 	)
 	(segment
+		(start 113.35 75.47)
+		(end 112.96 75.47)
+		(width 0.25)
+		(layer "F.Cu")
+		(net "Net-(D3-K)")
+	)
+	(segment
+		(start 121 83.12)
+		(end 113.35 75.47)
+		(width 0.25)
+		(layer "F.Cu")
+		(net "Net-(D3-K)")
+	)
+	(segment
 		(start 115.5 60.53)
 		(end 115.5 68)
@@
 		(net "Net-(D2-K)")
 	)
-	(segment
-		(start 113.35 75.47)
-		(end 112.96 75.47)
-		(width 0.25)
-		(layer "F.Cu")
-		(net "Net-(D3-K)")
-	)
-	(segment
-		(start 121 83.12)
-		(end 113.35 75.47)
-		(width 0.25)
-		(layer "F.Cu")
-		(net "Net-(D3-K)")
-	)
-	(segment
-		(start 101 63.020001)
-		(end 98.869999 60.89)
-		(width 0.25)
-		(layer "F.Cu")
-		(net "Net-(U1-PA6)")
-	)
-	(segment
-		(start 101 71.64)
-		(end 101 63.020001)
-		(width 0.25)
-		(layer "F.Cu")
-		(net "Net-(U1-PA6)")
-	)
-	(segment
-		(start 98.869999 60.89)
-		(end 97.845 60.89)
-		(width 0.25)
-		(layer "F.Cu")
-		(net "Net-(U1-PA6)")
-	)
-	(segment
-		(start 99.5 60.5)
-		(end 99.5 57.710001)
-		(width 0.25)
-		(layer "F.Cu")
-		(net "+3V3")
-	)
-	(segment
-		(start 100.634092 73)
-		(end 96 68.365908)
-		(width 0.25)
-		(layer "F.Cu")
-		(net "+3V3")
-	)
-	(segment
-		(start 105.1 71.64)
-		(end 105.1 65.6)
-		(width 0.25)
-		(layer "F.Cu")
-		(net "+3V3")
-	)
-	(segment
-		(start 99.5 57.710001)
-		(end 98.869999 57.08)
-		(width 0.25)
-		(layer "F.Cu")
-		(net "+3V3")
-	)
-	(segment
-		(start 96 68.365908)
-		(end 96 57)
-		(width 0.25)
-		(layer "F.Cu")
-		(net "+3V3")
-	)
-	(segment
-		(start 105.1 65.6)
-		(end 100 60.5)
-		(width 0.25)
-		(layer "F.Cu")
-		(net "+3V3")
-	)
-	(segment
-		(start 100 60.5)
-		(end 99.5 60.5)
-		(width 0.25)
-		(layer "F.Cu")
-		(net "+3V3")
-	)
-	(segment
-		(start 96.08 57.08)
-		(end 97.845 57.08)
-		(width 0.25)
-		(layer "F.Cu")
-		(net "+3V3")
-	)
-	(segment
-		(start 101 73)
-		(end 100.634092 73)
-		(width 0.25)
-		(layer "F.Cu")
-		(net "+3V3")
-	)
-	(segment
-		(start 96 57)
-		(end 96.08 57.08)
-		(width 0.25)
-		(layer "F.Cu")
-		(net "+3V3")
-	)
-	(segment
-		(start 98.869999 57.08)
-		(end 97.845 57.08)
-		(width 0.25)
-		(layer "F.Cu")
-		(net "+3V3")
-	)
 	(zone
